Commit message: add RGB-D camera

File: src/my_robot/urdf/my_robot.xacro (robot description, xacro)
@@ -47,4 +47,9 @@
         <parent link = "chassis"/>
         <child  link = "hokuyo"/>
+    </joint>
+    <joint name="camera_optical_joint" type="fixed">
+        <origin xyz = "0 0 0" rpy = "-1.5707 0 -1.5707"/>
+        <parent link = "camera_link"/>
+        <child  link = "camera_link_optical"/>
     </joint>
     <xacro:include filename = "$(find my_robot)/urdf/my_robot.gazebo"/>
@@ -157,4 +162,6 @@
         </inertial>
     </link>
+    <link name  = "cameral_ink_optical">
+    </link>
     <link name = "hokuyo">
         <visual>

Commit message: configure the rtabmap parameters for mapping.launch

File: src/my_robot/urdf/my_robot.xacro (robot description, xacro)
@@ -50,5 +50,5 @@
     <joint name="camera_optical_joint" type="fixed">
         <origin xyz = "0 0 0" rpy = "-1.5707 0 -1.5707"/>
-        <parent link = "camera_link"/>
+        <parent link = "camera"/>
         <child  link = "camera_link_optical"/>
     </joint>
@@ -162,5 +162,5 @@
         </inertial>
     </link>
-    <link name  = "cameral_ink_optical">
+    <link name  = "camera_link_optical">
     </link>
     <link name = "hokuyo">
